File: Microcontroller/ATmega328P.sch (EAGLE design)
At the start: 74 parts, among them IC2 7805T, IC7 ATMEGA168-20P, IC9 LM358N

Commit message: atmega schematic updated
Parts:
- removed C10, C24: 104, rcl:C-EU050-024X044
- removed C13, C15, C18, C3: (no value), rcl:CPOL-EUTT2D6
- removed C14, C26, C36, C5: (no value), rcl:C-EU050-024X044
- removed C17, C20, C25, C4: (no value), resistor:CPOL-EUE2.5-6
- removed C19, C22: (no value), resistor:C-EU050-024X044
- removed C23: 105, rcl:C-EU050-024X044
- removed D1, D2, D4, D6: (no value), adafruit:SCHOTTKY-DIODEDO41
- removed D7: (no value), diode:ZENER-DIODEDO35Z10
- removed HALL: CURRENT-SENSOR-ACS712#IC, diy-modules:CURRENT-SENSOR-ACS712#IC
- removed IC2: 7805T, linear:7805T
- removed IC3: (no value), linear:LM2596TH
- removed IC9: LM358N, linear:LM358N
- removed J2: (no value), con-amp:MTA02-100
- removed J5: (no value), con-amp:MTA03-100
- removed JP1: (no value), pinhead:PINHD-1X8
- removed JP7: (no value), adafruit:PINHD-1X6
- removed L3: (no value), rcl:L-EU0207/10
- removed R13, R14, R15, R17, R18, R25, R26, R27, R32, R33, R34, R37, R4, R51, R52, R53, R54, R55, R56, R7: (no value), rcl:R-EU_0204/7
- removed R23: 10K, 1%, rcl:R-EU_0204/7
- removed R24, R38, R45: 10k, 1%, rcl:R-EU_0204/7
- removed R46: 10k, rcl:R-EU_0207/12
- removed R49: 1, resistor:R-EU_MELF0207R
- removed R5: (no value), rcl:R-EU_0207/12
- removed R50: (no value), resistor:R-EU_MELF0207R
- removed VR1: K431, v-reg:TL431CLP
- removed X1: (no value), con-ptr500:AK500/10
- C1, C29: value (none) -> 100nF
- C28, C7: value (none) -> 22pF
- C9: value (none) -> 10nF
- IC7: value ATMEGA168-20P -> ATMEGA328P
- L2: value (none) -> 100mH
- Q2: value (none) -> 16MHz
- R61: value 2.2K -> 10k
Connections:
- removed net +12V: C17.+, C19.1, C4.+, D1.C, IC3.IN, R13.2, R14.2, R15.2, R17.2, R7.2
- removed net ADC0: JP7.2
- removed net ADC1: HALL.OUT, JP7.3
- removed net ADC2: C10.1, IC9A.OUT, JP7.4, R38.1
- removed net ADC3: C26.2, D7.C, JP7.5, R26.1
- removed net CH1-I: HALL.IN+, R24.2, R49.1, R50.1, X1-5.KL, X1-7.KL, X1-9.KL
- removed net E_PIN2: JP1.5
- removed net E_PIN3: JP1.4
- removed net E_PIN4: JP1.3, R5.2
- removed net N$12: HALL.VCC, R27.2, R32.2
- removed net N$13: HALL.GND, R33.2, R34.2
- removed net N$25: R25.1, R26.2, R37.2, R51.1, R52.1, R53.1, R54.2, R55.2, R56.2
- removed net N$29: D2.C, IC3.OUT, L3.2
- removed net N$31: IC3.FB, R18.2, R4.1
- removed net N$5: D1.A, J2.2, X1-1.KL
- removed net N$54: D4.A, D6.C
- removed net N$55: C10.2, IC9A.-IN, R23.1, R38.2
- removed net N$56: C24.1, J5.1, R46.2, VR1.C, VR1.R
- removed net N$60: C23.1, IC9A.+IN, R24.1, R45.1
- removed net N$63: C23.2, J5.2, R45.2
- removed net N$66: J2.1, R25.2, R51.2, R52.2, R53.2, X1-3.KL
- removed net N$7: C13.+, C15.+, C5.2, IC2.VI, R13.1, R14.1, R15.1, R17.1, R7.1
- removed net N$8: IC3.EN, R5.1
- removed net SIM_POW: C20.+, C22.1, C25.+, D4.C, JP1.1, L3.1, R4.2
- net GND: no longer C13.-, C14.1, C15.-, C17.-, C18.-, C19.2, C20.-, C22.2, C24.2, C25.-, C26.1, C3.-, C36.1, C4.-, C5.1, D2.A, D7.A, HALL.IN-, IC2.GND, IC3.GND, IC9P.V-, J5.3, JP1.2, JP1.7, JP7.1, R18.1, R23.2, R27.1, R33.1, R37.1, R49.2, R50.2, R54.1, R55.1, R56.1, VR1.A, X1-10.KL, X1-2.KL, X1-4.KL, X1-6.KL, X1-8.KL
- net VCC: no longer C14.2, C18.+, C3.+, C36.2, D6.A, IC2.VO, IC9P.V+, JP1.8, JP7.6, R32.1, R34.1, R46.1
