File: Microcontroller/MSP430FR2433_SMD_0402.sch (EAGLE design)
At the start: 11 parts, among them IC2 MSP430FR2433IRGET, Q1 32.768

Commit message: msp430fr2433 basic circuit complete
Connections:
- net N$13 renamed P2.2
- net N$14 renamed P3.0
Changed lines of the file:
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@@
 <setting verticaltext="up"/>
 </settings>
-<grid distance="0.05" unitdist="inch" unit="inch" style="lines" multiple="1" display="no" altdistance="0.01" altunitdist="inch" altunit="inch"/>
+<grid distance="0.1" unitdist="inch" unit="inch" style="lines" multiple="1" display="no" altdistance="0.01" altunitdist="inch" altunit="inch"/>
 <layers>
 <layer number="1" name="Top" color="4" fill="1" visible="no" active="no"/>
@@
 </segment>
 </net>
-<net name="N$13" class="0">
+<net name="P2.2" class="0">
 <segment>
 <pinref part="IC2" gate="G$1" pin="P2.2/ACLK"/>
 <wire x1="149.86" y1="109.22" x2="144.78" y2="109.22" width="0.1524" layer="91"/>
-</segment>
-</net>
-<net name="N$14" class="0">
+<label x="144.78" y="109.22" size="0.8128" layer="95" rot="R180" xref="yes"/>
+</segment>
+</net>
+<net name="P3.0" class="0">
 <segment>
 <pinref part="IC2" gate="G$1" pin="P3.0"/>
 <wire x1="149.86" y1="106.68" x2="144.78" y2="106.68" width="0.1524" layer="91"/>
-</segment>
-</net>
+<label x="144.78" y="106.68" size="0.8128" layer="95" rot="R180" xref="yes"/>
+</segment>
+</net>

Commit message: updated lot of ckt
Parts:
- removed J2: (no value), con-amp:MTA06-100
- removed Q1: 32.768, crystal:CRYTALTC26H
- added JP1, JP3: (no value), pinhead:PINHD-1X2
- added JP2: (no value), pinhead:PINHD-1X3
- added X1: 32.768KHZ, adafruit:XTAL-3.2X1.5
Connections:
- net GND: now also JP2.3, JP3.1; no longer J2.5
- net MSP_RST: now also JP1.1; no longer J2.1
- net N$1: now also X1.P$1; no longer Q1.1
- net N$3: now also X1.P$2; no longer Q1.2
- net RXD_A0: now also JP2.2; no longer J2.3
- net TEST: now also JP1.2; no longer J2.2
- net TXD_A0: now also JP2.1; no longer J2.4
- net VCC: now also JP3.2; no longer J2.6
Other:
- moved on the sheet: C3
