File: Memory/FLASH.sch (EAGLE design)
At the start: 2 parts, among them IC2 25AA040P

Commit message: vcc updated in the circuit
Parts:
- IC2: value 25AA040P -> W25Q64
Connections:
- new net VCC: C1.2, IC2.!WP, IC2.VCC
- net MISO: no longer C1.2, IC2.!WP, IC2.VCC
