File: Misc/Button_Led_Buzzer.sch (EAGLE design)
At the start: 4 parts

Commit message: few ckt updated
Parts:
- added BUZ1: F/TMB, buzzer:F/TMB
- added R2: 100K, resistor:R-US_0204/7
- added R3: 1K, resistor:R-US_0204/7
- added T1: (no value), transistor:BC547-NPN-TO92-CBE
- R12, R60: device resistor:R-US_R0805 -> resistor:R-US_0204/7
- renumbered POW to LED1, SETUP1 to BUTTON1
Connections:
- new net N$1: R2.2, R3.1, T1.B
- new net N$2: R3.2
- new net N$20: BUZ1.-, T1.C
- net GND: now also R2.1, T1.E
- net VCC: now also BUZ1.+
