File: RF/NRF24L01_Module_AnTenna.sch (EAGLE design)
At the start: 4 parts, among them M2 WIRELESS-NRF24L01-PA-EXT

Commit message: few ckt updated
Connections:
- net 3V3 renamed VCC
Changed lines of the file:
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@@
 <setting verticaltext="up"/>
 </settings>
-<grid distance="0.05" unitdist="inch" unit="inch" style="lines" multiple="1" display="no" altdistance="0.01" altunitdist="inch" altunit="inch"/>
+<grid distance="0.1" unitdist="inch" unit="inch" style="lines" multiple="1" display="no" altdistance="0.01" altunitdist="inch" altunit="inch"/>
 <layers>
 <layer number="1" name="Top" color="4" fill="1" visible="no" active="no"/>
@@
 <part name="C22" library="rcl" deviceset="C-EU" device="050-024X044" value="100nF"/>
 <part name="C23" library="rcl" deviceset="C-EU" device="050-024X044" value="1uF"/>
-<part name="U$1" library="PatternAgents-Beautify" deviceset="3V3" device=""/>
 <part name="M2" library="diy-modules" deviceset="WIRELESS-NRF24L01-PA-EXT" device=""/>
 <part name="C19" library="rcl" deviceset="C-EU" device="050-024X044" value="10nF"/>
+<part name="P+1" library="supply1" deviceset="VCC" device=""/>
 </parts>
 <sheets>
@@
 <attribute name="VALUE" x="-159.004" y="211.709" size="1.778" layer="96" rot="R180"/>
 </instance>
-<instance part="U$1" gate="G$1" x="-157.48" y="218.44"/>
 <instance part="M2" gate="G$1" x="-104.14" y="208.28"/>
 <instance part="C19" gate="G$1" x="-142.24" y="207.01" smashed="yes" rot="R180">
@@
 <attribute name="VALUE" x="-143.764" y="211.709" size="1.778" layer="96" rot="R180"/>
 </instance>
+<instance part="P+1" gate="VCC" x="-157.48" y="220.98"/>
 </instances>
 <busses>
@@
 </segment>
 </net>
-<net name="3V3" class="0">
-<segment>
-<pinref part="U$1" gate="G$1" pin="3V3"/>
+<net name="MISO" class="0">
+<segment>
+<wire x1="-127" y1="203.2" x2="-130.81" y2="203.2" width="0.1524" layer="91"/>
+<label x="-130.81" y="203.2" size="0.8128" layer="95" rot="R180" xref="yes"/>
+<pinref part="M2" gate="G$1" pin="MISO"/>
+</segment>
+</net>
+<net name="RF_CS" class="0">
+<segment>
+<wire x1="-127" y1="210.82" x2="-130.81" y2="210.82" width="0.1524" layer="91"/>
+<label x="-130.81" y="210.82" size="0.8128" layer="95" rot="R180" xref="yes"/>
+<pinref part="M2" gate="G$1" pin="CSN"/>
+</segment>
+</net>
+<net name="RF_IRQ" class="0">
+<segment>
+<pinref part="M2" gate="G$1" pin="IRQ"/>
+<wire x1="-127" y1="200.66" x2="-130.81" y2="200.66" width="0.1524" layer="91"/>
+<label x="-130.81" y="200.66" size="1.016" layer="95" rot="R180" xref="yes"/>
+</segment>
+</net>
+<net name="RF_CE" class="0">
+<segment>
+<wire x1="-127" y1="213.36" x2="-130.81" y2="213.36" width="0.1524" layer="91"/>
+<label x="-130.81" y="213.36" size="0.8128" layer="95" rot="R180" xref="yes"/>
+<pinref part="M2" gate="G$1" pin="CE"/>
+</segment>
+</net>
+<net name="VCC" class="0">
+<segment>
 <wire x1="-127" y1="215.9" x2="-142.24" y2="215.9" width="0.1524" layer="91"/>
 <wire x1="-142.24" y1="215.9" x2="-149.86" y2="215.9" width="0.1524" layer="91"/>
@@
 <wire x1="-142.24" y1="212.09" x2="-142.24" y2="215.9" width="0.1524" layer="91"/>
 <junction x="-142.24" y="215.9"/>
-</segment>
-</net>
-<net name="MISO" class="0">
-<segment>
-<wire x1="-127" y1="203.2" x2="-130.81" y2="203.2" width="0.1524" layer="91"/>
-<label x="-130.81" y="203.2" size="0.8128" layer="95" rot="R180" xref="yes"/>
-<pinref part="M2" gate="G$1" pin="MISO"/>
-</segment>
-</net>
-<net name="RF_CS" class="0">
-<segment>
-<wire x1="-127" y1="210.82" x2="-130.81" y2="210.82" width="0.1524" layer="91"/>
-<label x="-130.81" y="210.82" size="0.8128" layer="95" rot="R180" xref="yes"/>
-<pinref part="M2" gate="G$1" pin="CSN"/>
-</segment>
-</net>
-<net name="RF_IRQ" class="0">
-<segment>
-<pinref part="M2" gate="G$1" pin="IRQ"/>
-<wire x1="-127" y1="200.66" x2="-130.81" y2="200.66" width="0.1524" layer="91"/>
-<label x="-130.81" y="200.66" size="1.016" layer="95" rot="R180" xref="yes"/>
-</segment>
-</net>
-<net name="RF_CE" class="0">
-<segment>
-<wire x1="-127" y1="213.36" x2="-130.81" y2="213.36" width="0.1524" layer="91"/>
-<label x="-130.81" y="213.36" size="0.8128" layer="95" rot="R180" xref="yes"/>
-<pinref part="M2" gate="G$1" pin="CE"/>
-</segment>
-</net>
+<pinref part="P+1" gate="VCC" pin="VCC"/>
+</segment>
+</net>
