File: RF/SIM800L.sch (EAGLE design)
At the start: 12 parts, among them IC2 LM1117-adj

Commit message: few ckt updated
Parts:
- C1, C24, C26: device rcl:C-EUC0805 -> rcl:C-EU050-024X044
- C25: device rcl:CPOL-USUD-6,3X7,7 -> rcl:CPOL-USE2.5-6
Changed lines of the file:
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@@
 <setting verticaltext="up"/>
 </settings>
-<grid distance="0.05" unitdist="inch" unit="inch" style="lines" multiple="1" display="no" altdistance="0.01" altunitdist="inch" altunit="inch"/>
+<grid distance="0.1" unitdist="inch" unit="inch" style="lines" multiple="1" display="no" altdistance="0.01" altunitdist="inch" altunit="inch"/>
 <layers>
 <layer number="1" name="Top" color="4" fill="1" visible="yes" active="no"/>
@@
 <part name="GND1" library="supply1" deviceset="GND" device=""/>
 <part name="IC2" library="v-reg" deviceset="LD117A?*" device="S" technology="25TR" value="LM1117-adj"/>
-<part name="C1" library="rcl" deviceset="C-EU" device="C0805" value="100nF"/>
-<part name="C24" library="rcl" deviceset="C-EU" device="C0805" value="100nF"/>
+<part name="C1" library="rcl" deviceset="C-EU" device="050-024X044" value="100nF"/>
+<part name="C24" library="rcl" deviceset="C-EU" device="050-024X044" value="100nF"/>
 <part name="R11" library="resistor" deviceset="R-US_" device="0204/7" value="100k"/>
 <part name="R12" library="resistor" deviceset="R-US_" device="0204/7" value="43k"/>
 <part name="GND20" library="supply1" deviceset="GND" device=""/>
-<part name="C25" library="rcl" deviceset="CPOL-US" device="UD-6,3X7,7" value="220uF"/>
+<part name="C25" library="rcl" deviceset="CPOL-US" device="E2.5-6" value="220uF"/>
 <part name="P+13" library="supply1" deviceset="VCC" device=""/>
-<part name="C26" library="rcl" deviceset="C-EU" device="C0805" value="100nF"/>
+<part name="C26" library="rcl" deviceset="C-EU" device="050-024X044" value="100nF"/>
 <part name="C28" library="rcl" deviceset="CPOL-US" device="E2.5-6" value="100uF"/>
 <part name="R13" library="resistor" deviceset="R-US_" device="0204/7" value="1K"/>
