File: RF SOC/ESP8266_SMD_0603.sch (EAGLE design)
At the start: 34 parts, among them J1 DNP, Q1 600mA/40V, Q2 600mA/40V, U1 ESP8266, U3 W25Q32FV, U4 AP2112K-3.3V, Y1 26MHz

Commit message: Add files via upload
Parts:
- removed J3: (no value), con-amp:MTA02-100
Connections:
- net GND: no longer J3.2
- net VIN: no longer J3.1
Other:
- moved on the sheet: R17, R7, R9, U3

Commit message: esp8266 updated
Parts:
- removed C11: 0.1Uf, rcl:C-EUC0603
- removed C5, C7: 1uF, rcl:C-EUC0603
- removed C9: 0.1uF, rcl:C-EUC0603
- removed U4: AP2112K-3.3V, SparkFun-PowerIC:V_REG_LDOSMD
Connections:
- removed net VIN: C5.1, C9.1, U4.EN, U4.IN
- net GND: no longer C11.2, C5.2, C7.2, C9.2, U4.GND
- net VCC: no longer C11.1, C7.1, U4.OUT
Other:
- note removed: "ESP8266_CPU"
- note removed: "LDO"
- note removed: "VCC Range: 1.7V->3.6V"
- moved on the sheet: C1, C2, Q1, Q2, R17, R2, R4, R7, R9, U3
