File: Sensor/lis3dh 402/lis3dh v402.sch (EAGLE design)
At the start: 7 parts, among them U5 LIS3DHTR

Commit message: lis3dh 402 added
Parts:
- C17, C19: device rcl@1:C-EUC0603 -> rcl:C-EUC0402
- R11, R12: device rcl@1:R-US_R0603 -> rcl-2:R-US_R0402
Changed lines of the file:
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@@
 <part name="U$3" library="microbuilder" deviceset="GND" device=""/>
 <part name="U$30" library="microbuilder" deviceset="3.3V" device=""/>
-<part name="C17" library="rcl@1" deviceset="C-EU" device="C0603" value="0.1uF"/>
+<part name="C17" library="rcl" deviceset="C-EU" device="C0402" value="0.1uF"/>
 <part name="U$31" library="microbuilder" deviceset="GND" device=""/>
-<part name="C19" library="rcl@1" deviceset="C-EU" device="C0603" value="10µF"/>
+<part name="C19" library="rcl" deviceset="C-EU" device="C0402" value="10µF"/>
 <part name="U$36" library="microbuilder" deviceset="GND" device=""/>
-<part name="R11" library="rcl@1" deviceset="R-US_" device="R0603" value="10k"/>
+<part name="R11" library="rcl-2" deviceset="R-US_" device="R0402" value="10k"/>
 <part name="U$33" library="microbuilder" deviceset="3.3V" device=""/>
-<part name="R12" library="rcl@1" deviceset="R-US_" device="R0603" value="10k"/>
+<part name="R12" library="rcl-2" deviceset="R-US_" device="R0402" value="10k"/>
 <part name="SJ5" library="microbuilder" deviceset="SOLDERJUMPER_CLOSED" device=""/>
 <part name="SJ6" library="microbuilder" deviceset="SOLDERJUMPER_CLOSED" device=""/>
